File: pcb/bleep-pannel-pcb/bleep-pannel-pcb.kicad_pcb (KiCad board)
At the start: 2 copper layers, 80.3 x 36.8 mm, 23 parts, among them J1 CON_LED

Commit message: Updates and cover
Parts:
- J1: footprint Connector_PinHeader_2.54mm:PinHeader_1x02_P2.54mm_Vertical -> Connector_PinHeader_2.54mm:PinHeader_1x02_P2.54mm_Horizontal
- moved J1 2.22 mm to (69.7, 17.6), turned to 0 degrees
Routing:
- net Net-(D1-A): track 6.46 -> 11.1 mm
- net Net-(R_OC_OUT1-Pad1): track 8.83 -> 9.95 mm
- net Net-(D1-K): track 6.46 -> 7.33 mm

Commit message: Change LED handling
Parts:
- removed D1: LED, LED_THT:LED_D5.0mm
- removed J1: CON_LED, Connector_PinHeader_2.54mm:PinHeader_1x02_P2.54mm_Horizontal
- CON_SW1: footprint Connector_Wire:SolderWire-0.75sqmm_1x01_D1.25mm_OD3.5mm -> Connector_PinHeader_2.54mm:PinHeader_1x01_P2.54mm_Vertical
Routing:
- net Net-(D1-A): track 11.1 -> 0.00 mm
- net Net-(D1-K): track 7.33 -> 0.00 mm
