File: pcb/access-control-wroom-32e/access-control-wroom-32e.kicad_sch (KiCad schematic)
At the start: 31 parts, among them J1 CON_I2C, K1 G5LE-1, U1 ESP32-DevKitC

Commit message: Add values for refernce
Parts:
- R_T_LED1, R_T_RELAY1: value R -> 560R
Changed lines of the file:
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@@
 			)
 		)
-		(property "Value" "R"
+		(property "Value" "560R"
 			(at 201.93 72.3899 0)
 			(effects
@@
 			)
 		)
-		(property "Value" "R"
+		(property "Value" "560R"
 			(at 205.74 110.4899 0)
 			(effects

Commit message: Refined access controll dev box
Parts:
- added CON_AUX1: Conn_01x04_Socket, Connector_PinHeader_2.54mm:PinHeader_1x04_P2.54mm_Vertical, symbol Connector:Conn_01x04_Socket
- added C_SNUB1: C, Capacitor_THT:CP_Axial_L10.0mm_D6.0mm_P15.00mm_Horizontal, symbol Device:C
- added D_Z_3v3: D_Zener, Diode_THT:D_T-1_P10.16mm_Horizontal, symbol Device:D_Zener
- added J_NEUT1, J_NEUT2: Conn_01x01_Socket, Connector_Wire:SolderWire-2.5sqmm_1x01_D2.4mm_OD4.4mm, symbol Connector:Conn_01x01_Socket
- added RV_SNUB1: Varistor, Varistor:RV_Disc_D12mm_W3.9mm_P7.5mm, symbol Device:Varistor
- added R_SNUB1: R, Resistor_THT:R_Axial_DIN0617_L17.0mm_D6.0mm_P20.32mm_Horizontal, symbol Device:R
- C_5V_De1, C_5V_Med1: footprint Capacitor_THT:C_Disc_D3.4mm_W2.1mm_P2.50mm -> Capacitor_THT:C_Axial_L5.1mm_D3.1mm_P10.00mm_Horizontal
Connections:
- net +3V3: now also CON_AUX1.1 (Pin_1), D_Z_3v3.1 (K)
- net GND: now also CON_AUX1.2 (Pin_2), D_Z_3v3.2 (A)
- net at J_RELAY_LAMP1.1 (Pin_1), J_RELAY_NO1.1 (Pin_1), K1.3: now also RV_SNUB1.1, R_SNUB1.1
- net at U1.7 (32K_XP/GPIO32/ADC1_CH4): now also CON_AUX1.4 (Pin_4)
- net at U1.8 (32K_XN/GPIO33/ADC1_CH5): now also CON_AUX1.3 (Pin_3)
- new net: C_SNUB1.1, R_SNUB1.2
- new net NEUT: C_SNUB1.2, J_NEUT1.1 (Pin_1), J_NEUT2.1 (Pin_1), RV_SNUB1.2

Commit message: Updates with AUX
Parts:
- added CON_AUX2: Conn_01x04_Socket, Connector_PinHeader_2.54mm:PinHeader_1x04_P2.54mm_Vertical, symbol Connector:Conn_01x04_Socket
Connections:
- net +3V3: now also CON_AUX2.1 (Pin_1)
- net GND: now also CON_AUX2.2 (Pin_2)
- net at U1.29 (GPIO5): now also CON_AUX2.3 (Pin_3)
- net at U1.30 (GPIO18): now also CON_AUX2.4 (Pin_4)
Changed lines of the file:
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@@
+	)
+	(junction
+		(at 172.72 39.37)
+		(diameter 0)
+		(color 0 0 0 0)
 	)
 	(junction
@@
 	)
 	(junction
+		(at 180.34 35.56)
+		(diameter 0)
+		(color 0 0 0 0)
+	)
+	(junction
 		(at 213.36 30.48)
 		(diameter 0)
@@
 	)
 	(junction
+		(at 166.37 63.5)
+		(diameter 0)
+		(color 0 0 0 0)
+	)
+	(junction
 		(at 215.9 59.69)
 		(diameter 0)
@@
 	(wire
 		(pts
+			(xy 182.88 55.88) (xy 187.96 55.88)
+		)
+		(stroke
+			(width 0)
+			(type default)
+		)
+	)
+	(wire
+		(pts
 			(xy 199.39 74.93) (xy 199.39 83.82)
 		)
@@
 	(wire
 		(pts
+			(xy 187.96 63.5) (xy 187.96 58.42)
+		)
+		(stroke
+			(width 0)
+			(type default)
+		)
+	)
+	(wire
+		(pts
 			(xy 222.25 78.74) (xy 228.6 78.74)
 		)
@@
 	(wire
 		(pts
+			(xy 162.56 63.5) (xy 166.37 63.5)
+		)
+		(stroke
+			(width 0)
+			(type default)
+		)
+	)
+	(wire
+		(pts
 			(xy 157.48 59.69) (xy 215.9 59.69)
 		)
@@
 	(wire
 		(pts
+			(xy 162.56 64.77) (xy 162.56 63.5)
+		)
+		(stroke
+			(width 0)
+			(type default)
+		)
+	)
+	(wire
+		(pts
 			(xy 91.44 54.61) (xy 74.93 54.61)
 		)
@@
 	(wire
 		(pts
+			(xy 172.72 50.8) (xy 172.72 39.37)
+		)
+		(stroke
+			(width 0)
+			(type default)
+		)
+	)
+	(wire
+		(pts
 			(xy 215.9 67.31) (xy 215.9 69.85)
 		)
@@
 	(wire
 		(pts
+			(xy 157.48 64.77) (xy 162.56 64.77)
+		)
+		(stroke
+			(width 0)
+			(type default)
+		)
+	)
+	(wire
+		(pts
 			(xy 220.98 60.96) (xy 220.98 63.5)
 		)
@@
 	(wire
 		(pts
+			(xy 187.96 50.8) (xy 172.72 50.8)
+		)
+		(stroke
+			(width 0)
+			(type default)
+		)
+	)
+	(wire
+		(pts
 			(xy 157.48 72.39) (xy 167.64 72.39)
 		)
@@
 	(wire
 		(pts
+			(xy 187.96 53.34) (xy 195.58 53.34)
+		)
+		(stroke
+			(width 0)
+			(type default)
+		)
+	)
+	(wire
+		(pts
 			(xy 176.53 48.26) (xy 176.53 49.53)
 		)
@@
 	(wire
 		(pts
-			(xy 168.91 39.37) (xy 177.8 39.37)
+			(xy 168.91 39.37) (xy 172.72 39.37)
 		)
 		(stroke
@@
 	(wire
 		(pts
+			(xy 166.37 63.5) (xy 187.96 63.5)
+		)
+		(stroke
+			(width 0)
+			(type default)
+		)
+	)
+	(wire
+		(pts
 			(xy 113.03 39.37) (xy 118.11 39.37)
 		)
@@
 	(wire
 		(pts
+			(xy 166.37 64.77) (xy 166.37 63.5)
+		)
+		(stroke
+			(width 0)
+			(type default)
+		)
+	)
+	(wire
+		(pts
 			(xy 144.78 27.94) (xy 154.94 27.94)
 		)
@@
 	(wire
 		(pts
+			(xy 172.72 39.37) (xy 177.8 39.37)
+		)
+		(stroke
+			(width 0)
+			(type default)
+		)
+	)
+	(wire
+		(pts
 			(xy 289.56 73.66) (xy 295.91 73.66)
 		)
@@
 	(wire
 		(pts
+			(xy 182.88 62.23) (xy 182.88 55.88)
+		)
+		(stroke
+			(width 0)
+			(type default)
+		)
+	)
+	(wire
+		(pts
 			(xy 276.86 81.28) (xy 287.02 81.28)
 		)
@@
 	(wire
 		(pts
+			(xy 195.58 35.56) (xy 180.34 35.56)
+		)
+		(stroke
+			(width 0)
+			(type default)
+		)
+	)
+	(wire
+		(pts
 			(xy 124.46 34.29) (xy 124.46 36.83)
 		)
@@
 	(wire
 		(pts
+			(xy 157.48 62.23) (xy 182.88 62.23)
+		)
+		(stroke
+			(width 0)
+			(type default)
+		)
+	)
+	(wire
+		(pts
 			(xy 105.41 29.21) (xy 118.11 29.21)
 		)
@@
 		(pts
 			(xy 74.93 54.61) (xy 74.93 48.26)
+		)
+		(stroke
+			(width 0)
+			(type default)
+		)
+	)
+	(wire
+		(pts
+			(xy 195.58 53.34) (xy 195.58 35.56)
 		)
 		(stroke
@@
 					(unit 1)
 				)
+			)
+		)
+	)
+	(symbol
+		(lib_id "Connector:Conn_01x04_Socket")
+		(at 193.04 53.34 0)
+		(unit 1)
+		(exclude_from_sim no)
+		(in_bom yes)
+		(on_board yes)
+		(dnp no)
+		(fields_autoplaced yes)
+		(property "Reference" "CON_AUX2"
+			(at 194.31 53.3399 0)
+			(effects
+				(font
+					(size 1.27 1.27)
+				)
+				(justify left)
+			)
+		)
+		(property "Value" "Conn_01x04_Socket"
+			(at 194.31 55.8799 0)
+			(effects
+				(font
+					(size 1.27 1.27)
+				)
+				(justify left)
+			)
+		)
+		(property "Footprint" "Connector_PinHeader_2.54mm:PinHeader_1x04_P2.54mm_Vertical"
+			(at 193.04 53.34 0)
+			(effects
+				(font
+					(size 1.27 1.27)
+				)
+				(hide yes)
+			)
+		)
+		(property "Datasheet" "~"
+			(at 193.04 53.34 0)
+			(effects
+				(font
+					(size 1.27 1.27)
+				)
+				(hide yes)
+			)
+		)
+		(property "Description" "Generic connector, single row, 01x04, script generated"
+			(at 193.04 53.34 0)
+			(effects
+				(font
+					(size 1.27 1.27)
+				)
+				(hide yes)
+			)
+		)
+		(pin "2"
+		)
+		(pin "1"
+		)
+		(pin "4"
+		)
+		(pin "3"
+		)
+		(instances
+			(project "access-control-wroom-32e"
+				(path "/79724983-fbb7-47f3-9f65-a8afc53dd20f"
+					(reference "CON_AUX2")
+					(unit 1)
+				)

Commit message: Further optimisation
Parts:
- added CON_SENSE1: Conn_01x04_Socket, Connector_PinHeader_2.54mm:PinHeader_1x04_P2.54mm_Vertical, symbol Connector:Conn_01x04_Socket
Connections:
- net +3V3: now also CON_SENSE1.1 (Pin_1)
- net +5V: now also CON_SENSE1.4 (Pin_4)
- net GND: now also CON_SENSE1.2 (Pin_2)
- net at U1.13 (MTDI/GPIO12/ADC2_CH5): now also CON_SENSE1.3 (Pin_3)
