File: pcb/current-sensor-pcb/current-sensor-pcb.kicad_sch (KiCad schematic)
At the start: 12 parts, among them U1 TLI4971A050T5UE0001XUMA1

Commit message: Progress with SMT controller and contactor variant
Parts:
- added C_3V3_1, C_3V3_2, C_AOUT1: C, Capacitor_THT:C_Disc_D3.8mm_W2.6mm_P2.50mm, symbol Device:C
- added J_LV_IN2, J_LV_OUT2: Conn_01x01_Socket, Connector_Wire:SolderWirePad_1x01_SMD_5x10mm, symbol Connector:Conn_01x01_Socket
Connections:
- net +3V3: now also C_3V3_1.1, C_3V3_2.1
- net GND: now also C_3V3_1.2, C_3V3_2.2, C_AOUT1.2
- net at R_OC_LV1.1: now also U_OC1.2; no longer U_OC1.1
- net at J_LV_OUT1.1 (Pin_1), R_OC_LV1.2, U1.7 (IP-): now also J_LV_OUT2.1 (Pin_1)
- net at J_CON_SENSE1.3 (Pin_3), U1.4 (AOUT): now also C_AOUT1.1
- net at J_LV_IN1.1 (Pin_1), U1.8 (IP+): now also J_LV_IN2.1 (Pin_1)
- net at R_OC_NEUT1.1: now also U_OC1.1; no longer U_OC1.2
Other:
- moved on the sheet: J_LV_IN1, J_LV_OUT1, J_NE1, R_OC_LV1, R_OC_NEUT1

Commit message: Slight refactor of contator components to support more compact layout
Connections:
- net at R_OC_LV1.1: now also U_OC1.1; no longer U_OC1.2
- net at R_OC_NEUT1.1: now also U_OC1.2; no longer U_OC1.1
Other:
- moved on the sheet: J_NE1, R_OC_LV1, R_OC_NEUT1
Changed lines of the file:
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@@
+	(wire
+		(pts
+			(xy 113.03 101.6) (xy 113.03 102.87)
+		)
+		(stroke
+			(width 0)
+			(type default)
+		)
+	)
 	(wire
 		(pts
@@
 	(wire
 		(pts
+			(xy 113.03 113.03) (xy 104.14 113.03)
+		)
+		(stroke
+			(width 0)
+			(type default)
+		)
+	)
+	(wire
+		(pts
 			(xy 165.1 30.48) (xy 165.1 31.75)
 		)
@@
 	(wire
 		(pts
-			(xy 72.39 60.96) (xy 72.39 107.95)
+			(xy 72.39 60.96) (xy 72.39 101.6)
 		)
 		(stroke
@@
 	(wire
 		(pts
-			(xy 99.06 95.25) (xy 105.41 95.25)
-		)
-		(stroke
-			(width 0)
-			(type default)
-		)
-	)
-	(wire
-		(pts
-			(xy 113.03 95.25) (xy 113.03 102.87)
+			(xy 90.17 113.03) (xy 96.52 113.03)
 		)
 		(stroke
@@
 	(wire
 		(pts
-			(xy 72.39 107.95) (xy 97.79 107.95)
+			(xy 72.39 101.6) (xy 78.74 101.6)
 		)
 		(stroke
@@
 	(wire
 		(pts
-			(xy 105.41 107.95) (xy 113.03 107.95)
+			(xy 113.03 107.95) (xy 113.03 113.03)
+		)
+		(stroke
+			(width 0)
+			(type default)
+		)
+	)
+	(wire
+		(pts
+			(xy 86.36 101.6) (xy 113.03 101.6)
 		)
 		(stroke
@@
 	(symbol
 		(lib_id "Connector:Conn_01x01_Socket")
-		(at 93.98 95.25 180)
+		(at 85.09 113.03 180)
 		(unit 1)
 		(exclude_from_sim no)
@@
 		(fields_autoplaced yes)
 		(property "Reference" "J_NE1"
-			(at 94.615 90.17 0)
+			(at 85.725 107.95 0)
 			(effects
 				(font
@@
 		)
 		(property "Value" "Conn_01x01_Socket"
-			(at 94.615 92.71 0)
+			(at 85.725 110.49 0)
 			(effects
 				(font
@@
 		)
 		(property "Footprint" "Connector_Wire:SolderWire-2.5sqmm_1x01_D2.4mm_OD3.6mm"
-			(at 93.98 95.25 0)
+			(at 85.09 113.03 0)
 			(effects
 				(font
@@
 		)
 		(property "Datasheet" "~"
-			(at 93.98 95.25 0)
+			(at 85.09 113.03 0)
 			(effects
 				(font
@@
 		)
 		(property "Description" "Generic connector, single row, 01x01, script generated"
-			(at 93.98 95.25 0)
+			(at 85.09 113.03 0)
 			(effects
 				(font
@@
 	(symbol
 		(lib_id "Device:R")
-		(at 101.6 107.95 270)
+		(at 82.55 101.6 270)
 		(unit 1)
 		(exclude_from_sim no)
@@
 		(fields_autoplaced yes)
 		(property "Reference" "R_OC_LV1"
-			(at 101.6 101.6 90)
+			(at 82.55 95.25 90)
 			(effects
 				(font
@@
 		)
 		(property "Value" "100KR"
-			(at 101.6 104.14 90)
+			(at 82.55 97.79 90)
 			(effects
 				(font
@@
 		)
 		(property "Footprint" "Resistor_THT:R_Axial_DIN0617_L17.0mm_D6.0mm_P20.32mm_Horizontal"
-			(at 101.6 106.172 90)
+			(at 82.55 99.822 90)
 			(effects
 				(font
@@
 		)
 		(property "Datasheet" "~"
-			(at 101.6 107.95 0)
+			(at 82.55 101.6 0)
 			(effects
 				(font
@@
 		)
 		(property "Description" "Resistor"
-			(at 101.6 107.95 0)
+			(at 82.55 101.6 0)
 			(effects
 				(font
@@
 	(symbol
 		(lib_id "Device:R")
-		(at 109.22 95.25 270)
+		(at 100.33 113.03 270)
 		(unit 1)
 		(exclude_from_sim no)
@@
 		(fields_autoplaced yes)
 		(property "Reference" "R_OC_NEUT1"
-			(at 109.22 88.9 90)
+			(at 100.33 106.68 90)
 			(effects
 				(font
@@
 		)
 		(property "Value" "100KR"
-			(at 109.22 91.44 90)
+			(at 100.33 109.22 90)
 			(effects
 				(font
@@
 		)
 		(property "Footprint" "Resistor_THT:R_Axial_DIN0617_L17.0mm_D6.0mm_P20.32mm_Horizontal"
-			(at 109.22 93.472 90)
+			(at 100.33 111.252 90)
 			(effects
 				(font
@@
 		)
 		(property "Datasheet" "~"
-			(at 109.22 95.25 0)
+			(at 100.33 113.03 0)
 			(effects
 				(font
@@
 		)
 		(property "Description" "Resistor"
-			(at 109.22 95.25 0)
-			(effects
-				(font
+			(at 100.33 113.03 0)
+			(effects
+				(font

Commit message: Final changes pre manufacture
Parts:
- added J_NE2: Conn_01x01_Socket, Connector_Wire:SolderWire-2.5sqmm_1x01_D2.4mm_OD3.6mm, symbol Connector:Conn_01x01_Socket
Connections:
- net at J_NE1.1 (Pin_1), R_OC_NEUT1.2: now also J_NE2.1 (Pin_1)
Changed lines of the file:
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@@
+	)
+	(junction
+		(at 90.17 113.03)
+		(diameter 0)
+		(color 0 0 0 0)
 	)
 	(junction
@@
 		(pts
 			(xy 123.19 26.67) (xy 130.81 26.67)
+		)
+		(stroke
+			(width 0)
+			(type default)
+		)
+	)
+	(wire
+		(pts
+			(xy 90.17 113.03) (xy 90.17 118.11)
 		)
 		(stroke
@@
 					(unit 1)
 				)
+			)
+		)
+	)
+	(symbol
+		(lib_id "Connector:Conn_01x01_Socket")
+		(at 85.09 118.11 180)
+		(unit 1)
+		(exclude_from_sim no)
+		(in_bom yes)
+		(on_board yes)
+		(dnp no)
+		(fields_autoplaced yes)
+		(property "Reference" "J_NE2"
+			(at 85.725 113.03 0)
+			(effects
+				(font
+					(size 1.27 1.27)
+				)
+			)
+		)
+		(property "Value" "Conn_01x01_Socket"
+			(at 85.725 115.57 0)
+			(effects
+				(font
+					(size 1.27 1.27)
+				)
+			)
+		)
+		(property "Footprint" "Connector_Wire:SolderWire-2.5sqmm_1x01_D2.4mm_OD3.6mm"
+			(at 85.09 118.11 0)
+			(effects
+				(font
+					(size 1.27 1.27)
+				)
+				(hide yes)
+			)
+		)
+		(property "Datasheet" "~"
+			(at 85.09 118.11 0)
+			(effects
+				(font
+					(size 1.27 1.27)
+				)
+				(hide yes)
+			)
+		)
+		(property "Description" "Generic connector, single row, 01x01, script generated"
+			(at 85.09 118.11 0)
+			(effects
+				(font
+					(size 1.27 1.27)
+				)
+				(hide yes)
+			)
+		)
+		(pin "1"
+		)
+		(instances
+			(project "current-sensor-pcb"
+				(path "/ed885ae9-e2ca-4fb3-ad41-8083aa76f12b"
+					(reference "J_NE2")
+					(unit 1)
+				)
