File: pcb/access-control-devkitc-relay/access-control-devkitc-relay.kicad_sch (KiCad schematic)
At the start: 12 parts, among them K1 G5LE-1

Commit message: Update with values
Parts:
- added D3: D_Zener, Diode_THT:D_DO-41_SOD81_P10.16mm_Horizontal, symbol Device:D_Zener
- renumbered J_COIL_HIGH to J_COIL_HIGH1, J_COIL_LOW to J_COIL_LOW1
Connections:
- net at J_COIL_LOW1.1 (Pin_1), K1.2: now also D3.1 (K); no longer D1.2 (A)
- new net: D1.2 (A), D3.2 (A)
Other:
- moved on the sheet: C_SNUB1, D1, J_COIL_HIGH1, J_COIL_LOW1, J_NEUT1, J_NEUT2, J_RELAY_COM1, J_RELAY_LAMP1, J_RELAY_NO1, K1, RV_SNUB1, R_SNUB1

Commit message: Fixes to relief, JST connectors for SMT board
Parts:
- added J_NEUT3, J_RELAY_LAMP2: Conn_01x01_Socket, Connector_Wire:SolderWire-2.5sqmm_1x01_D2.4mm_OD4.4mm, symbol Connector:Conn_01x01_Socket
Connections:
- net NEUT: now also J_NEUT3.1 (Pin_1)
- net at J_RELAY_LAMP1.1 (Pin_1), J_RELAY_NO1.1 (Pin_1), K1.3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: now also J_RELAY_LAMP2.1 (Pin_1)
Changed lines of the file:
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@@
+	)
+	(junction
+		(at 236.22 91.44)
+		(diameter 0)
+		(color 0 0 0 0)
 	)
 	(junction
@@
 		(pts
 			(xy 236.22 73.66) (xy 236.22 87.63)
+		)
+		(stroke
+			(width 0)
+			(type default)
+		)
+	)
+	(wire
+		(pts
+			(xy 205.74 88.9) (xy 205.74 92.71)
+		)
+		(stroke
+			(width 0)
+			(type default)
+		)
+	)
+	(wire
+		(pts
+			(xy 236.22 91.44) (xy 236.22 95.25)
 		)
 		(stroke
@@
 	(symbol
 		(lib_id "Connector:Conn_01x01_Socket")
+		(at 210.82 92.71 0)
+		(unit 1)
+		(exclude_from_sim no)
+		(in_bom yes)
+		(on_board yes)
+		(dnp no)
+		(fields_autoplaced yes)
+		(property "Reference" "J_RELAY_LAMP2"
+			(at 212.09 91.4399 0)
+			(effects
+				(font
+					(size 1.27 1.27)
+				)
+				(justify left)
+			)
+		)
+		(property "Value" "Conn_01x01_Socket"
+			(at 212.09 93.9799 0)
+			(effects
+				(font
+					(size 1.27 1.27)
+				)
+				(justify left)
+			)
+		)
+		(property "Footprint" "Connector_Wire:SolderWire-2.5sqmm_1x01_D2.4mm_OD4.4mm"
+			(at 210.82 92.71 0)
+			(effects
+				(font
+					(size 1.27 1.27)
+				)
+				(hide yes)
+			)
+		)
+		(property "Datasheet" "~"
+			(at 210.82 92.71 0)
+			(effects
+				(font
+					(size 1.27 1.27)
+				)
+				(hide yes)
+			)
+		)
+		(property "Description" "Generic connector, single row, 01x01, script generated"
+			(at 210.82 92.71 0)
+			(effects
+				(font
+					(size 1.27 1.27)
+				)
+				(hide yes)
+			)
+		)
+		(pin "1"
+		)
+		(instances
+			(project "access-control-devkitc-relay"
+				(path "/79724983-fbb7-47f3-9f65-a8afc53dd20f"
+					(reference "J_RELAY_LAMP2")
+					(unit 1)
+				)
+			)
+		)
+	)
+	(symbol
+		(lib_id "Connector:Conn_01x01_Socket")
 		(at 241.3 87.63 0)
 		(unit 1)
@@
 					(unit 1)
 				)
+			)
+		)
+	)
+	(symbol
+		(lib_id "Connector:Conn_01x01_Socket")
+		(at 241.3 95.25 0)
+		(unit 1)
+		(exclude_from_sim no)
+		(in_bom yes)
+		(on_board yes)
+		(dnp no)
+		(fields_autoplaced yes)
+		(property "Reference" "J_NEUT3"
+			(at 242.57 93.9799 0)
+			(effects
+				(font
+					(size 1.27 1.27)
+				)
+				(justify left)
+			)
+		)
+		(property "Value" "Conn_01x01_Socket"
+			(at 242.57 96.5199 0)
+			(effects
+				(font
+					(size 1.27 1.27)
+				)
+				(justify left)
+			)
+		)
+		(property "Footprint" "Connector_Wire:SolderWire-2.5sqmm_1x01_D2.4mm_OD4.4mm"
+			(at 241.3 95.25 0)
+			(effects
+				(font
+					(size 1.27 1.27)
+				)
+				(hide yes)
+			)
+		)
+		(property "Datasheet" "~"
+			(at 241.3 95.25 0)
+			(effects
+				(font
+					(size 1.27 1.27)
+				)
+				(hide yes)
+			)
+		)
+		(property "Description" "Generic connector, single row, 01x01, script generated"
+			(at 241.3 95.25 0)
+			(effects
+				(font
+					(size 1.27 1.27)
+				)
+				(hide yes)
+			)
+		)
+		(pin "1"
+		)
+		(instances
+			(project "access-control-devkitc-relay"
+				(path "/79724983-fbb7-47f3-9f65-a8afc53dd20f"
+					(reference "J_NEUT3")
+					(unit 1)
+				)

Commit message: Final changes pre manufacture
Parts:
- added CON_DAISY1: Conn_01x04_Socket, Connector_JST:JST_XA_B04B-XASK-1_1x04_P2.50mm_Vertical, symbol Connector:Conn_01x04_Socket
- added CON_MCU1: Conn_01x04_Socket, Connector_PinHeader_2.54mm:PinHeader_1x04_P2.54mm_Vertical, symbol Connector:Conn_01x04_Socket
- added CON_PWR1: Conn_01x02_Socket, Connector_JST:JST_XH_B2B-XH-A_1x02_P2.50mm_Vertical, symbol Connector:Conn_01x02_Socket
- added C_5V_Large1: 1000uf, Capacitor_THT:CP_Radial_D8.0mm_P5.00mm, symbol Device:C_Polarized
- added JP1: SolderJumper_2_Open, Jumper:SolderJumper-2_P1.3mm_Open_TrianglePad1.0x1.5mm, symbol Jumper:SolderJumper_2_Open
Connections:
- net +5V: now also CON_DAISY1.2 (Pin_2), CON_MCU1.2 (Pin_2), CON_PWR1.2 (Pin_2), C_5V_Large1.1
- net at D3.1 (K), J_COIL_LOW1.1 (Pin_1), K1.2: now also CON_DAISY1.3 (Pin_3), JP1.2 (B)
- new net: CON_MCU1.3 (Pin_3), JP1.1 (A)
- new net: CON_DAISY1.4 (Pin_4), CON_MCU1.4 (Pin_4)
- new net GND: CON_DAISY1.1 (Pin_1), CON_MCU1.1 (Pin_1), CON_PWR1.1 (Pin_1), C_5V_Large1.2
