File: pcb/access-control-devkitc-psu/access-control-devkitc-psu.kicad_pcb (KiCad board)
At the start: 2 copper layers, 38.5 x 40.5 mm, 5 parts, among them J1 Conn_01x02_Socket

Commit message: Option for 5v out on the other side
Parts:
- added J2: Conn_01x02_Socket, Connector_PinHeader_2.54mm:PinHeader_1x02_P2.54mm_Vertical, F.Cu at (36.1, 34.9)
Routing:
- net Net-(J1-Pin_1): track 12.6 -> 40.5 mm
- net Net-(J1-Pin_2): track 25.2 -> 46.2 mm

Commit message: Commit to transfer SMT PSU
Routing:
- net Net-(J1-Pin_2): track 46.2 -> 46.8 mm
- net (no net): vias 0 -> 2
Changed lines of the file:
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@@
 		(layer "Edge.Cuts")
+	)
+	(via
+		(at 2.5 2.5)
+		(size 3.5)
+		(drill 3)
+		(layers "F.Cu" "B.Cu")
+		(net 0)
+	)
+	(via
+		(at 30 35.5)
+		(size 3.5)
+		(drill 3)
+		(layers "F.Cu" "B.Cu")
+		(free yes)
+		(net 0)
 	)
 	(segment
@@
 	)
 	(segment
-		(start 36.11 37.39)
-		(end 16.61 37.39)
+		(start 15.5 38.5)
+		(end 18 36)
 		(width 2)
 		(layer "F.Cu")
@@
 	)
 	(segment
-		(start 15.5 38.5)
-		(end 18 36)
+		(start 34.5 39)
+		(end 36.11 37.39)
 		(width 2)
 		(layer "F.Cu")
@@
 	)
 	(segment
+		(start 20.4 36)
+		(end 23.4 39)
+		(width 2)
+		(layer "F.Cu")
+		(net 1)
+	)
+	(segment
 		(start 4.46 37.46)
 		(end 6 39)
 		(width 2)
 		(layer "F.Cu")
+		(net 1)
+	)
+	(segment
+		(start 23.4 39)
+		(end 34.5 39)
+		(width 2)
+		(layer "F.Cu")
+		(net 1)
+	)
+	(segment
+		(start 18 36)
+		(end 20.4 36)
+		(width 2)
+		(layer "F.Cu")
